File: BE-Carrier-Example.brd (EAGLE design)
At the start: 50 x 50 mm, 1 part

Commit message: Updated BlackEdge Carrier Drawing
Parts:
- U$1: value BE-CARRIERSMD -> BE-CARRIER; device BlackEdge:BE-CARRIER-SMD -> BlackEdge:BE-CARRIER
Changed lines of the file:
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@@
 </autorouter>
 <elements>
-<element name="U$1" library="BlackEdge" package="BE-CARRIER-SMD" value="BE-CARRIERSMD" x="25" y="25"/>
+<element name="U$1" library="BlackEdge" package="BE-CARRIER" value="BE-CARRIER" x="25" y="25"/>
 </elements>
 <signals>
